Commit message: [ros2]: adding ros2 cart...

File: ros/pkgs/uwbcart_ros/urdf/cubeBot.gazebo.xacro (robot description, xacro)
@@ -92,5 +92,5 @@
     </plugin>
   </gazebo>
-<!--link : https://www.raspberrypi.org/documentation/hardware/camera/-->
+<!--link  https://www.raspberrypi.org/documentation/hardware/camera/-->
   <gazebo reference="camera_rgb_frame">
     <sensor type="camera" name="Pi Camera">

File: ros2/pkgs/uwbcart_ros/urdf/cubeBot.urdf.xacro (robot description, xacro)
@@ -13,5 +13,5 @@
       <origin xyz="0 0 0.0" rpy="0 0 0"/>
       <geometry>
-        <mesh filename="package://uwbcart_ros/models/cubeBot/meshes/main.dae" scale="1 1 1"/>
+        <mesh filename="file://$(find uwbcart_ros)/models/cubeBot/meshes/main.dae" scale="1 1 1"/>
       </geometry>
     </visual>
@@ -40,5 +40,5 @@
       <origin xyz="0 0 0" rpy="1.57 0 0"/>
       <geometry>
-        <mesh filename="package://uwbcart_ros/models/cubeBot/meshes/wheel.stl" scale="1 1 1"/>
+        <mesh filename="ile://$(find uwbcart_ros)/models/cubeBot/meshes/wheel.stl" scale="1 1 1"/>
       </geometry>
       <material name="dark"/>
@@ -68,5 +68,5 @@
       <origin xyz="0 0 0" rpy="1.57 0 0"/>
       <geometry>
-        <mesh filename="package://uwbcart_ros/models/cubeBot/meshes/wheel.stl" scale="1 1 1"/>
+        <mesh filename="ile://$(find uwbcart_ros)/models/cubeBot/meshes/wheel.stl" scale="1 1 1"/>
       </geometry>
       <material name="dark"/>
