Commit message: [ros2]:cubeBot showed in ros2 gazebo.

File: ros2/pkgs/uwbcart_ros/urdf/cubeBot.urdf.xacro (robot description, xacro)
@@ -40,5 +40,5 @@
       <origin xyz="0 0 0" rpy="1.57 0 0"/>
       <geometry>
-        <mesh filename="ile://$(find uwbcart_ros)/models/cubeBot/meshes/wheel.stl" scale="1 1 1"/>
+        <mesh filename="file://$(find uwbcart_ros)/models/cubeBot/meshes/wheel.stl" scale="1 1 1"/>
       </geometry>
       <material name="dark"/>
@@ -68,5 +68,5 @@
       <origin xyz="0 0 0" rpy="1.57 0 0"/>
       <geometry>
-        <mesh filename="ile://$(find uwbcart_ros)/models/cubeBot/meshes/wheel.stl" scale="1 1 1"/>
+        <mesh filename="file://$(find uwbcart_ros)/models/cubeBot/meshes/wheel.stl" scale="1 1 1"/>
       </geometry>
       <material name="dark"/>

Commit message: [ros2]: modify bot

File: ros2/pkgs/uwbcart_ros/urdf/cubeBot.urdf.xacro (robot description, xacro)
@@ -33,5 +33,5 @@
     <parent link="base_link"/>
     <child link="wheel_left_link"/>
-    <origin xyz="0.0 0.040 0.005" rpy="-1.57 0 0"/>
+    <origin xyz="0.0 0.0785 0.005" rpy="-1.57 0 0"/>
     <axis xyz="0 0 1"/>
   </joint>
@@ -61,5 +61,5 @@
     <parent link="base_link"/>
     <child link="wheel_right_link"/>
-    <origin xyz="0.0 -0.040 0.005" rpy="-1.57 0 0"/>
+    <origin xyz="0.0 -0.0785 0.005" rpy="-1.57 0 0"/>
     <axis xyz="0 0 1"/>
   </joint>
