Commit message: [ros2]: rename cubeBot --> cart.

File: ros2/pkgs/uwbcart_ros/urdf/cart.urdf.xacro (robot description, xacro)
@@ -1,6 +1,6 @@
 <?xml version="1.0" ?>
-<robot name="cubeBot" xmlns:xacro="http://ros.org/wiki/xacro">
-  <xacro:include filename="$(find uwbcart_ros)/urdf/cubeBot_mat.xacro"/>
-  <xacro:include filename="$(find uwbcart_ros)/urdf/cubeBot.gazebo.xacro"/>
+<robot name="cart" xmlns:xacro="http://ros.org/wiki/xacro">
+  <xacro:include filename="$(find uwbcart_ros)/urdf/cart_mat.xacro"/>
+  <xacro:include filename="$(find uwbcart_ros)/urdf/cart.gazebo.xacro"/>
   <link name="base_footprint"/>
   <joint name="base_joint" type="fixed">
@@ -13,5 +13,5 @@
       <origin xyz="0 0 0.0" rpy="0 0 0"/>
       <geometry>
-        <mesh filename="file://$(find uwbcart_ros)/models/cubeBot/meshes/main.dae" scale="1 1 1"/>
+        <mesh filename="file://$(find uwbcart_ros)/models/cart/meshes/main.dae" scale="1 1 1"/>
       </geometry>
     </visual>
@@ -40,5 +40,5 @@
       <origin xyz="0 0 0" rpy="1.57 0 0"/>
       <geometry>
-        <mesh filename="file://$(find uwbcart_ros)/models/cubeBot/meshes/wheel.stl" scale="1 1 1"/>
+        <mesh filename="file://$(find uwbcart_ros)/models/cart/meshes/wheel.stl" scale="1 1 1"/>
       </geometry>
       <material name="dark"/>
@@ -68,5 +68,5 @@
       <origin xyz="0 0 0" rpy="1.57 0 0"/>
       <geometry>
-        <mesh filename="file://$(find uwbcart_ros)/models/cubeBot/meshes/wheel.stl" scale="1 1 1"/>
+        <mesh filename="file://$(find uwbcart_ros)/models/cart/meshes/wheel.stl" scale="1 1 1"/>
       </geometry>
       <material name="dark"/>
